File: simulation/binary_conversion/antimax.sch (KiCad schematic (older format))
At the start: 6 parts, among them M10 2N7002, M7 2N7002, M8 BSS84, M9 BSS84

Commit message: ternary adders, switches, and cyclers
Changed lines of the file:
@@
 $Descr A4 11693 8268
 encoding utf-8
-Sheet 65 64
+Sheet 10 91
 Title ""
 Date ""
@@
 AR Path="/639E88A2/5FCD1DE6/5FCD23BD" Ref="M?"  Part="1"
 AR Path="/639E88A8/5FCD1DE6/5FCD23BD" Ref="M6"  Part="1"
-F 0 "M6" H 5988 3246 50  0000 L CNN
+F 0 "M102" H 5988 3246 50  0000 L CNN
 F 1 "BSS84" H 5988 3155 50  0000 L CNN
 F 2 "" H 5700 3200 50  0001 C CNN
@@
 AR Path="/639E88A2/5FCD1DE6/5FCD44CC" Ref="M?"  Part="1"
 AR Path="/639E88A8/5FCD1DE6/5FCD44CC" Ref="M7"  Part="1"
-F 0 "M7" H 5988 3946 50  0000 L CNN
+F 0 "M103" H 5988 3946 50  0000 L CNN
 F 1 "BSS84" H 5988 3855 50  0000 L CNN
 F 2 "" H 5700 3900 50  0001 C CNN
@@
 AR Path="/639E88A2/5FCD1DE6/5FCD4EDA" Ref="M?"  Part="1"
 AR Path="/639E88A8/5FCD1DE6/5FCD4EDA" Ref="M8"  Part="1"
-F 0 "M8" H 5988 5046 50  0000 L CNN
+F 0 "M104" H 5988 5046 50  0000 L CNN
 F 1 "2N7002" H 5988 4955 50  0000 L CNN
 F 2 "" H 5675 5000 50  0001 C CNN
@@
 AR Path="/639E88A2/5FCD1DE6/5FCD5EC6" Ref="M?"  Part="1"
 AR Path="/639E88A8/5FCD1DE6/5FCD5EC6" Ref="M5"  Part="1"
-F 0 "M5" H 5138 5046 50  0000 L CNN
+F 0 "M101" H 5138 5046 50  0000 L CNN
 F 1 "2N7002" H 5138 4955 50  0000 L CNN
 F 2 "" H 4825 5000 50  0001 C CNN
@@
 AR Path="/639E88A2/5FCD1DE6/5FCD72D0" Ref="R?"  Part="1"
 AR Path="/639E88A8/5FCD1DE6/5FCD72D0" Ref="R5"  Part="1"
-F 0 "R5" H 5870 4296 50  0000 L CNN
+F 0 "R17" H 5870 4296 50  0000 L CNN
 F 1 "12k" H 5870 4205 50  0000 L CNN
 F 2 "" V 5730 4250 50  0001 C CNN
@@
 AR Path="/639E88A2/5FCD1DE6/5FCD771F" Ref="R?"  Part="1"
 AR Path="/639E88A8/5FCD1DE6/5FCD771F" Ref="R6"  Part="1"
-F 0 "R6" H 5870 4696 50  0000 L CNN
+F 0 "R18" H 5870 4696 50  0000 L CNN
 F 1 "12k" H 5870 4605 50  0000 L CNN
 F 2 "" V 5730 4650 50  0001 C CNN
