File: simulation/binary_conversion/and.sch (KiCad schematic (older format))
At the start: 0 parts

Commit message: ternary adders, switches, and cyclers
Changed lines of the file:
@@
 $Descr A4 11693 8268
 encoding utf-8
-Sheet 38 64
+Sheet 89 91
 Title ""
 Date ""
@@
 Text HLabel 8350 3650 2    50   Output ~ 0
 Out
+$Sheet
+S 7050 3500 550  300
+U 60DA9D23
+F0 "Sheet60DA9D22" 50
+F1 "nand.sch" 50
+F2 "A" I L 7050 3550 50
+F3 "B" I L 7050 3650 50
+F4 "Out" O R 7600 3650 50
+F5 "C" I L 7050 3750 50
+$EndSheet
 $EndSCHEMATC
