File: simulation/binary_conversion/nand.sch (KiCad schematic (older format))
At the start: 6 parts, among them M105 MPMOS, M106 MPMOS, M107 MPMOS, M108 MNMOS, M109 MNMOS, M110 MNMOS

Commit message: ternary adders, switches, and cyclers
Parts:
- M105, M106, M107: value MPMOS -> BSS84
- M108, M109, M110: value MNMOS -> 2N7002

Commit message: update readme.md to include current project status
Changed lines of the file:
@@
 AR Path="/5FEFC423/60DA9D23/5FD23F99" Ref="M307"  Part="1"
 AR Path="/5FEE09C6/60DA9D23/5FD23F99" Ref="M313"  Part="1"
-F 0 "M313" H 7138 5046 50  0000 L CNN
+F 0 "M217" H 7138 5046 50  0000 L CNN
 F 1 "2N7002" H 7138 4955 50  0000 L CNN
 F 2 "" H 6825 5000 50  0001 C CNN
@@
 AR Path="/5FEFC423/60DA9D23/5FD25BD8" Ref="M308"  Part="1"
 AR Path="/5FEE09C6/60DA9D23/5FD25BD8" Ref="M314"  Part="1"
-F 0 "M314" H 7138 5546 50  0000 L CNN
+F 0 "M218" H 7138 5546 50  0000 L CNN
 F 1 "2N7002" H 7138 5455 50  0000 L CNN
 F 2 "" H 6825 5500 50  0001 C CNN
@@
 AR Path="/5FEFC423/60DA9D23/5FD261AE" Ref="M306"  Part="1"
 AR Path="/5FEE09C6/60DA9D23/5FD261AE" Ref="M312"  Part="1"
-F 0 "M312" H 7138 4546 50  0000 L CNN
+F 0 "M216" H 7138 4546 50  0000 L CNN
 F 1 "BSS84" H 7138 4455 50  0000 L CNN
 F 2 "" H 6850 4500 50  0001 C CNN
@@
 AR Path="/5FEFC423/60DA9D23/5FD265C9" Ref="M305"  Part="1"
 AR Path="/5FEE09C6/60DA9D23/5FD265C9" Ref="M311"  Part="1"
-F 0 "M311" H 6338 4546 50  0000 L CNN
+F 0 "M215" H 6338 4546 50  0000 L CNN
 F 1 "BSS84" H 6338 4455 50  0000 L CNN
 F 2 "" H 6050 4500 50  0001 C CNN
@@
 AR Path="/5FEFC423/60DA9D23/5FE9BEF2" Ref="#PWR0131"  Part="1"
 AR Path="/5FEE09C6/60DA9D23/5FE9BEF2" Ref="#PWR0132"  Part="1"
-F 0 "#PWR0132" H 7000 6000 50  0001 C CNN
+F 0 "#PWR0116" H 7000 6000 50  0001 C CNN
 F 1 "GND" H 7005 6077 50  0000 C CNN
 F 2 "" H 7000 6250 50  0001 C CNN
@@
 AR Path="/5FEFC423/60DA9D23/5FEE325D" Ref="M304"  Part="1"
 AR Path="/5FEE09C6/60DA9D23/5FEE325D" Ref="M310"  Part="1"
-F 0 "M310" H 5588 4546 50  0000 L CNN
+F 0 "M214" H 5588 4546 50  0000 L CNN
 F 1 "BSS84" H 5588 4455 50  0000 L CNN
 F 2 "" H 5300 4500 50  0001 C CNN
@@
 AR Path="/5FEFC423/60DA9D23/5FEE63C8" Ref="M309"  Part="1"
 AR Path="/5FEE09C6/60DA9D23/5FEE63C8" Ref="M315"  Part="1"
-F 0 "M315" H 7138 6046 50  0000 L CNN
+F 0 "M219" H 7138 6046 50  0000 L CNN
 F 1 "2N7002" H 7138 5955 50  0000 L CNN
 F 2 "" H 6825 6000 50  0001 C CNN
