File: simulation/addition/nconsensus.sch (KiCad schematic (older format))
At the start: 6 parts, among them M1 MPMOS, M15 MPMOS, M16 MNMOS, M2 MNMOS

Commit message: remove nconensus gate from sum gate, removed .sch-bak and cache files
Changed lines of the file:
@@
 $Descr A4 11693 8268
 encoding utf-8
-Sheet 5 28
+Sheet 5 26
 Title ""
 Date ""
@@
 AR Path="/5FDE2F92/5FDD79FE/5FEDF3F0/600A1223/5FF3A517" Ref="M611"  Part="1"
 AR Path="/5FDE2F92/5FDD79FE/5FDC7A5D/5FF3A517" Ref="M621"  Part="1"
-F 0 "M131" H 5088 3196 50  0000 L CNN
+AR Path="/5FDC5271/600A11AC/5FF3A517" Ref="M3"  Part="1"
+AR Path="/5FDC5271/600A1223/5FF3A517" Ref="M?"  Part="1"
+F 0 "M3" H 5088 3196 50  0000 L CNN
 F 1 "MPMOS" H 5088 3105 50  0000 L CNN
 F 2 "" H 4800 3150 50  0001 C CNN
@@
 AR Path="/5FDE2F92/5FDD79FE/5FEDF3F0/600A1223/5FF3AEA3" Ref="M612"  Part="1"
 AR Path="/5FDE2F92/5FDD79FE/5FDC7A5D/5FF3AEA3" Ref="M622"  Part="1"
-F 0 "M132" H 5088 4296 50  0000 L CNN
+AR Path="/5FDC5271/600A11AC/5FF3AEA3" Ref="M4"  Part="1"
+AR Path="/5FDC5271/600A1223/5FF3AEA3" Ref="M?"  Part="1"
+F 0 "M4" H 5088 4296 50  0000 L CNN
 F 1 "MNMOS" H 5088 4205 50  0000 L CNN
 F 2 "" H 4775 4250 50  0001 C CNN
@@
 AR Path="/5FDE2F92/5FDD79FE/5FEDF3F0/600A1223/5FF438E6" Ref="R382"  Part="1"
 AR Path="/5FDE2F92/5FDD79FE/5FDC7A5D/5FF438E6" Ref="R390"  Part="1"
-F 0 "R82" H 4970 3946 50  0000 L CNN
+AR Path="/5FDC5271/600A11AC/5FF438E6" Ref="R3"  Part="1"
+AR Path="/5FDC5271/600A1223/5FF438E6" Ref="R?"  Part="1"
+F 0 "R3" H 4970 3946 50  0000 L CNN
 F 1 "12k" H 4970 3855 50  0000 L CNN
 F 2 "" V 4830 3900 50  0001 C CNN
@@
 AR Path="/5FDE2F92/5FDD79FE/5FEDF3F0/600A1223/5FF3F52B" Ref="R381"  Part="1"
 AR Path="/5FDE2F92/5FDD79FE/5FDC7A5D/5FF3F52B" Ref="R389"  Part="1"
-F 0 "R81" H 4970 3546 50  0000 L CNN
+AR Path="/5FDC5271/600A11AC/5FF3F52B" Ref="R2"  Part="1"
+AR Path="/5FDC5271/600A1223/5FF3F52B" Ref="R?"  Part="1"
+F 0 "R2" H 4970 3546 50  0000 L CNN
 F 1 "12k" H 4970 3455 50  0000 L CNN
 F 2 "" V 4830 3500 50  0001 C CNN
@@
 AR Path="/5FDE2F92/5FDD79FE/5FEDF3F0/600A1223/5FF39477" Ref="M609"  Part="1"
 AR Path="/5FDE2F92/5FDD79FE/5FDC7A5D/5FF39477" Ref="M619"  Part="1"
-F 0 "M129" H 4288 3196 50  0000 L CNN
+AR Path="/5FDC5271/600A11AC/5FF39477" Ref="M1"  Part="1"
+AR Path="/5FDC5271/600A1223/5FF39477" Ref="M?"  Part="1"
+F 0 "M1" H 4288 3196 50  0000 L CNN
 F 1 "MPMOS" H 4288 3105 50  0000 L CNN
 F 2 "" H 4000 3150 50  0001 C CNN
@@
 AR Path="/5FDE2F92/5FDD79FE/5FEDF3F0/600A1223/5FF3BB83" Ref="M610"  Part="1"
 AR Path="/5FDE2F92/5FDD79FE/5FDC7A5D/5FF3BB83" Ref="M620"  Part="1"
-F 0 "M130" H 4288 4296 50  0000 L CNN
+AR Path="/5FDC5271/600A11AC/5FF3BB83" Ref="M2"  Part="1"
+AR Path="/5FDC5271/600A1223/5FF3BB83" Ref="M?"  Part="1"
+F 0 "M2" H 4288 4296 50  0000 L CNN
 F 1 "MNMOS" H 4288 4205 50  0000 L CNN
 F 2 "" H 3975 4250 50  0001 C CNN

Commit message: lowered transistor count for sum gate
Changed lines of the file:
@@
 $Descr A4 11693 8268
 encoding utf-8
-Sheet 5 26
+Sheet 5 24
 Title ""
 Date ""
@@
 AR Path="/5FDC5271/600A11AC/5FF3A517" Ref="M3"  Part="1"
 AR Path="/5FDC5271/600A1223/5FF3A517" Ref="M?"  Part="1"
-F 0 "M3" H 5088 3196 50  0000 L CNN
+AR Path="/5FDCD92F/600A11AC/5FF3A517" Ref="M3"  Part="1"
+AR Path="/5FDD3C70/5FDA8800/5FEDF3F0/600A11AC/5FF3A517" Ref="M19"  Part="1"
+AR Path="/5FDD3C70/5FDA8800/5FDC7A5D/5FF3A517" Ref="M23"  Part="1"
+AR Path="/5FDD3C70/5FDD79FE/5FEDF3F0/600A11AC/5FF3A517" Ref="M45"  Part="1"
+AR Path="/5FDD3C70/5FDD79FE/5FDC7A5D/5FF3A517" Ref="M49"  Part="1"
+F 0 "M49" H 5088 3196 50  0000 L CNN
 F 1 "MPMOS" H 5088 3105 50  0000 L CNN
 F 2 "" H 4800 3150 50  0001 C CNN
@@
 AR Path="/5FDC5271/600A11AC/5FF3AEA3" Ref="M4"  Part="1"
 AR Path="/5FDC5271/600A1223/5FF3AEA3" Ref="M?"  Part="1"
-F 0 "M4" H 5088 4296 50  0000 L CNN
+AR Path="/5FDCD92F/600A11AC/5FF3AEA3" Ref="M4"  Part="1"
+AR Path="/5FDD3C70/5FDA8800/5FEDF3F0/600A11AC/5FF3AEA3" Ref="M20"  Part="1"
+AR Path="/5FDD3C70/5FDA8800/5FDC7A5D/5FF3AEA3" Ref="M24"  Part="1"
+AR Path="/5FDD3C70/5FDD79FE/5FEDF3F0/600A11AC/5FF3AEA3" Ref="M46"  Part="1"
+AR Path="/5FDD3C70/5FDD79FE/5FDC7A5D/5FF3AEA3" Ref="M50"  Part="1"
+F 0 "M50" H 5088 4296 50  0000 L CNN
 F 1 "MNMOS" H 5088 4205 50  0000 L CNN
 F 2 "" H 4775 4250 50  0001 C CNN
@@
 AR Path="/5FDC5271/600A11AC/5FF438E6" Ref="R3"  Part="1"
 AR Path="/5FDC5271/600A1223/5FF438E6" Ref="R?"  Part="1"
-F 0 "R3" H 4970 3946 50  0000 L CNN
+AR Path="/5FDCD92F/600A11AC/5FF438E6" Ref="R3"  Part="1"
+AR Path="/5FDD3C70/5FDA8800/5FEDF3F0/600A11AC/5FF438E6" Ref="R14"  Part="1"
+AR Path="/5FDD3C70/5FDA8800/5FDC7A5D/5FF438E6" Ref="R16"  Part="1"
+AR Path="/5FDD3C70/5FDD79FE/5FEDF3F0/600A11AC/5FF438E6" Ref="R30"  Part="1"
+AR Path="/5FDD3C70/5FDD79FE/5FDC7A5D/5FF438E6" Ref="R32"  Part="1"
+F 0 "R32" H 4970 3946 50  0000 L CNN
 F 1 "12k" H 4970 3855 50  0000 L CNN
 F 2 "" V 4830 3900 50  0001 C CNN
@@
 AR Path="/5FDC5271/600A11AC/5FF3F52B" Ref="R2"  Part="1"
 AR Path="/5FDC5271/600A1223/5FF3F52B" Ref="R?"  Part="1"
-F 0 "R2" H 4970 3546 50  0000 L CNN
+AR Path="/5FDCD92F/600A11AC/5FF3F52B" Ref="R1"  Part="1"
+AR Path="/5FDD3C70/5FDA8800/5FEDF3F0/600A11AC/5FF3F52B" Ref="R13"  Part="1"
+AR Path="/5FDD3C70/5FDA8800/5FDC7A5D/5FF3F52B" Ref="R15"  Part="1"
+AR Path="/5FDD3C70/5FDD79FE/5FEDF3F0/600A11AC/5FF3F52B" Ref="R29"  Part="1"
+AR Path="/5FDD3C70/5FDD79FE/5FDC7A5D/5FF3F52B" Ref="R31"  Part="1"
+F 0 "R31" H 4970 3546 50  0000 L CNN
 F 1 "12k" H 4970 3455 50  0000 L CNN
 F 2 "" V 4830 3500 50  0001 C CNN
@@
 AR Path="/5FDC5271/600A11AC/5FF39477" Ref="M1"  Part="1"
 AR Path="/5FDC5271/600A1223/5FF39477" Ref="M?"  Part="1"
-F 0 "M1" H 4288 3196 50  0000 L CNN
+AR Path="/5FDCD92F/600A11AC/5FF39477" Ref="M1"  Part="1"
+AR Path="/5FDD3C70/5FDA8800/5FEDF3F0/600A11AC/5FF39477" Ref="M17"  Part="1"
+AR Path="/5FDD3C70/5FDA8800/5FDC7A5D/5FF39477" Ref="M21"  Part="1"
+AR Path="/5FDD3C70/5FDD79FE/5FEDF3F0/600A11AC/5FF39477" Ref="M43"  Part="1"
+AR Path="/5FDD3C70/5FDD79FE/5FDC7A5D/5FF39477" Ref="M47"  Part="1"
+F 0 "M47" H 4288 3196 50  0000 L CNN
 F 1 "MPMOS" H 4288 3105 50  0000 L CNN
 F 2 "" H 4000 3150 50  0001 C CNN
@@
 AR Path="/5FDC5271/600A11AC/5FF3BB83" Ref="M2"  Part="1"
 AR Path="/5FDC5271/600A1223/5FF3BB83" Ref="M?"  Part="1"
-F 0 "M2" H 4288 4296 50  0000 L CNN
+AR Path="/5FDCD92F/600A11AC/5FF3BB83" Ref="M2"  Part="1"
+AR Path="/5FDD3C70/5FDA8800/5FEDF3F0/600A11AC/5FF3BB83" Ref="M18"  Part="1"
+AR Path="/5FDD3C70/5FDA8800/5FDC7A5D/5FF3BB83" Ref="M22"  Part="1"
+AR Path="/5FDD3C70/5FDD79FE/5FEDF3F0/600A11AC/5FF3BB83" Ref="M44"  Part="1"
+AR Path="/5FDD3C70/5FDD79FE/5FDC7A5D/5FF3BB83" Ref="M48"  Part="1"
+F 0 "M48" H 4288 4296 50  0000 L CNN
 F 1 "MNMOS" H 4288 4205 50  0000 L CNN
 F 2 "" H 3975 4250 50  0001 C CNN
