File: simulation/addition/addition.sch (KiCad schematic (older format))
At the start: 7 parts

Commit message: update readme.md to include current project status
Changed lines of the file:
@@
 $Descr A2 23386 16535
 encoding utf-8
-Sheet 1 6
+Sheet 1 2
 Title ""
 Date ""
@@
 $Sheet
 S 3350 4050 500  300
-U 5FDD3C70
-F0 "Sheet5FDD3C6F" 50
-F1 "full_adder.sch" 50
-F2 "A" I L 3350 4100 50
+U 5FE8E33C
+F0 "Sheet5FE8E33B" 50
+F1 "flat_schematic.sch" 50
+F2 "C" I L 3350 4300 50
 F3 "B" I L 3350 4200 50
-F4 "C" I L 3350 4300 50
+F4 "A" I L 3350 4100 50
 F5 "Sum" O R 3850 4150 50
 F6 "Carry" O R 3850 4250 50

Commit message: re-organized project directory and started work on ALU pcb
Parts:
- V3, V4: Spice_Model dc(-5) -> dc(5)
Changed lines of the file:
@@
 Text Notes 2550 3450 0    50   ~ 0
 Weird cases:\nii1 = Too many iterations\n011 = Too many iterations\n111 = Too many iterations
-Text GLabel 3350 4300 0    50   Input ~ 0
-C
-Text GLabel 3350 4200 0    50   Input ~ 0
-B
-Text GLabel 3350 4100 0    50   Input ~ 0
-A
 Text GLabel 4150 4250 2    50   Output ~ 0
 Carry
@@
 F 4 "Y" H 1300 3950 50  0001 L CNN "Spice_Netlist_Enabled"
 F 5 "V" H 1300 3950 50  0001 L CNN "Spice_Primitive"
-F 6 "dc(-5)" H 1430 3859 50  0000 L CNN "Spice_Model"
+F 6 "dc(5)" H 1430 3859 50  0000 L CNN "Spice_Model"
 	1    1300 3950
 	1    0    0    -1
@@
 F 4 "Y" H 900 3950 50  0001 L CNN "Spice_Netlist_Enabled"
 F 5 "V" H 900 3950 50  0001 L CNN "Spice_Primitive"
-F 6 "dc(-5)" H 1030 3859 50  0000 L CNN "Spice_Model"
+F 6 "dc(5)" H 1030 3859 50  0000 L CNN "Spice_Model"
 	1    900  3950
 	1    0    0    -1
 $EndComp
+Text GLabel 3350 4100 0    50   Input ~ 0
+A
+Text GLabel 3350 4200 0    50   Input ~ 0
+B
+Text GLabel 3350 4300 0    50   Input ~ 0
+C
 $Sheet
 S 3350 4050 500  300
-U 5FE8E33C
-F0 "Sheet5FE8E33B" 50
+U 5FFB596F
+F0 "Sheet5FFB596E" 50
 F1 "flat_schematic.sch" 50
 F2 "C" I L 3350 4300 50

Commit message: started pure ternary alu
Parts:
- V3: Spice_Model dc(5) -> dc(-5)
- V4: Spice_Model dc(5) -> dc(0)
Other:
- note added: "A B C | C S\n– – – | – 0\n– – 0 | – +\n– – + | 0 –\n– 0 – | – +\n– 0 0 | 0 –\n– 0 + | 0 0\n– + – | 0 –\n– + 0 | 0 0\n– + + | 0 +\n0 – – | – +\n0 – 0 | 0 –\n0 – + | 0 0\n0 0 – | 0 –\n0 0 0 | 0 0\n0 0 + | 0 +\n0 + – | 0 0\n0 + 0 | 0 +\n0 + + | + –\n+ – – | 0 –\n+ – 0 | 0 0\n+ – + | 0 +\n+ 0 – | 0 0\n+ 0 0 | 0 +\n+ 0 + | + –\n+ + – | 0 +\n+ + 0 | + –\n+ + + | + 0"
Changed lines of the file:
@@
 $Descr A2 23386 16535
 encoding utf-8
-Sheet 1 2
+Sheet 1 4
 Title ""
 Date ""
@@
 F 4 "Y" H 1300 3950 50  0001 L CNN "Spice_Netlist_Enabled"
 F 5 "V" H 1300 3950 50  0001 L CNN "Spice_Primitive"
-F 6 "dc(5)" H 1430 3859 50  0000 L CNN "Spice_Model"
+F 6 "dc(0)" H 1430 3859 50  0000 L CNN "Spice_Model"
 	1    1300 3950
 	1    0    0    -1
@@
 F 4 "Y" H 900 3950 50  0001 L CNN "Spice_Netlist_Enabled"
 F 5 "V" H 900 3950 50  0001 L CNN "Spice_Primitive"
-F 6 "dc(5)" H 1030 3859 50  0000 L CNN "Spice_Model"
+F 6 "dc(-5)" H 1030 3859 50  0000 L CNN "Spice_Model"
 	1    900  3950
 	1    0    0    -1
@@
 $Sheet
 S 3350 4050 500  300
-U 5FFB596F
-F0 "Sheet5FFB596E" 50
-F1 "flat_schematic.sch" 50
-F2 "C" I L 3350 4300 50
+U 5FF05F9A
+F0 "A+B+C" 50
+F1 "full_adder.sch" 50
+F2 "A" I L 3350 4100 50
 F3 "B" I L 3350 4200 50
-F4 "A" I L 3350 4100 50
+F4 "C" I L 3350 4300 50
 F5 "Sum" O R 3850 4150 50
 F6 "Carry" O R 3850 4250 50
 $EndSheet
+Text Notes 1500 2775 0    50   ~ 0
+A    B    C  |  C    S\n–    –    –  |  –    0\n–    –    0  |  –    +\n–    –    +  |  0    –\n–    0    –  |  –    +\n–    0    0  |  0    –\n–    0    +  |  0    0\n–    +    –  |  0    –\n–    +    0  |  0    0\n–    +    +  |  0    +\n0    –    –  |  –    +\n0    –    0  |  0    –\n0    –    +  |  0    0\n0    0    –  |  0    –\n0    0    0  |  0    0\n0    0    +  |  0    +\n0    +    –  |  0    0\n0    +    0  |  0    +\n0    +    +  |  +    –\n+    –    –  |  0    –\n+    –    0  |  0    0\n+    –    +  |  0    +\n+    0    –  |  0    0\n+    0    0  |  0    +\n+    0    +  |  +    –\n+    +    –  |  0    +\n+    +    0  |  +    –\n+    +    +  |  +    0
 $EndSCHEMATC
