File: simulation/addition/flat_schematic.sch (KiCad schematic (older format))
At the start: 94 parts

Commit message: update readme.md to include current project status
Parts:
- removed M? (x29): MPMOS, symbol pspice:MPMOS
- removed M? (x29): MNMOS, symbol pspice:MNMOS
- removed R? (x36): 12k, symbol Device:R
- added A1, A14, A16, A17, A6, A8, A9: nany, Ternary_Rev_1:nany, symbol addition-rescue:nany-Ternary
- added A10, A11, A2, A3: nconsensus, Ternary_Rev_1:nconsensus, symbol addition-rescue:nconsensus-Ternary
- added A12, A13, A15, A18, A4, A5, A7: inverter, Ternary_Rev_1:inverter, symbol addition-rescue:inverter-Ternary
Connections:
- wire segments 503 -> 61
Other:
- note removed: "A"
- note removed: "A\n"
- note removed: "B"
- note removed: "C"
- note removed: "Carry"
- note removed: "Carry\n"
- note removed: "In"
- note removed: "In\n"
- note removed: "Out"
- note removed: "Out\n"
- note removed: "Sum"
- note removed: "Sum\n"
- note removed: "full adder\n"
- note removed: "half adder\n"
- note removed: "inverter\n"
- note removed: "nany gate"
- note removed: "nconsensus gate\n"
- note removed: "sum gate"

Commit message: re-organized project directory and started work on ALU pcb
Parts:
- removed A1, A14, A16, A17, A6, A8, A9: nany, Ternary_Rev_1:nany, symbol addition-rescue:nany-Ternary
- removed A10, A11, A2, A3: nconsensus, Ternary_Rev_1:nconsensus, symbol addition-rescue:nconsensus-Ternary
- removed A12, A13, A15, A18, A4, A5, A7: inverter, Ternary_Rev_1:inverter, symbol addition-rescue:inverter-Ternary
- added A? (x7): nany, Ternary_Rev_1:nany, symbol Ternary:nany
- added A? (x4): nconsensus, Ternary_Rev_1:nconsensus, symbol Ternary:nconsensus
- added A? (x7): inverter, Ternary_Rev_1:inverter, symbol Ternary:inverter

Commit message: started pure ternary alu
Connections:
- wire segments 61 -> 64
