File: simulation/binary_encoding/binary_encoding.sch (KiCad schematic (older format))
At the start: 18 parts, among them M1 MPMOS, M2 MNMOS, M3 MPMOS, M4 MNMOS

Commit message: started pure ternary alu
Parts:
- removed D2, D3, D4: D, symbol Device:D
- removed M1, M3: MPMOS, symbol pspice:MPMOS
- removed M2, M4: MNMOS, symbol pspice:MNMOS
- added Q1, Q2, Q3, Q4, Q5: BSS8402DW, Package_TO_SOT_SMD:SOT-363_SC-70-6_Handsoldering, symbol Ternary:BSS8402DW
- added R8: 12k, symbol Device:R
- D1: Spice_Lib_File diode.lib -> /lab/dev/tritium/library/gates_spice.lib; Spice_Primitive D -> D
- R3, R4: value 10M -> 12M
- R7: value 10M -> 12k
- V1: Spice_Model dc(-5) -> dc(5)
- V2: Spice_Model dc(5) -> dc(-5)
Connections:
- net labels added: 1, In, Out, Vdd, Vss, i
- net labels removed: +5V, -5V, High, Low, Vin, Vout
- wire segments 47 -> 64
Other:
- note added: "Decoder"
- note added: "Encoder\n"
- moved on the sheet: V1, V2, V3
