File: pcbs/alu/alu.kicad_pcb (KiCad board)
At the start: 2 copper layers, 240 x 80.6 mm, 1038 parts, among them J1 Conn_02x20_Odd_Even, Q1 BSS8402DW, Q10 BSS8402DW, Q100 BSS8402DW, Q101 BSS8402DW, Q102 BSS8402DW, Q103 BSS8402DW, Q104 BSS8402DW, Q105 BSS8402DW, Q106 BSS8402DW, Q107 BSS8402DW, Q108 BSS8402DW, Q109 BSS8402DW, Q11 BSS8402DW, Q110 BSS8402DW, Q111 BSS8402DW, Q112 BSS8402DW, Q113 BSS8402DW, Q114 BSS8402DW, Q115 BSS8402DW, Q116 BSS8402DW, Q117 BSS8402DW, Q118 BSS8402DW, Q119 BSS8402DW, Q12 BSS8402DW, Q120 BSS8402DW, Q121 BSS8402DW, Q122 BSS8402DW, Q123 BSS8402DW, Q124 BSS8402DW, Q125 BSS8402DW, Q126 BSS8402DW, Q127 BSS8402DW, Q128 BSS8402DW, Q129 BSS8402DW, Q13 BSS8402DW, Q130 BSS8402DW, Q131 BSS8402DW, Q132 BSS8402DW, Q133 BSS8402DW, Q134 BSS8402DW, Q135 BSS8402DW, Q136 BSS8402DW, Q137 BSS8402DW, Q138 BSS8402DW, Q139 BSS8402DW, Q14 BSS8402DW, Q140 BSS8402DW, Q141 BSS8402DW, Q142 BSS8402DW, Q143 BSS8402DW, Q144 BSS8402DW, Q145 BSS8402DW, Q146 BSS8402DW, Q147 BSS8402DW, Q148 BSS8402DW, Q149 BSS8402DW, Q15 BSS8402DW, Q150 BSS8402DW, Q151 BSS8402DW, Q152 BSS8402DW, Q153 BSS8402DW, Q154 BSS8402DW, Q155 BSS8402DW, Q156 BSS8402DW, Q157 BSS8402DW, Q158 BSS8402DW, Q159 BSS8402DW, Q16 BSS8402DW, Q160 BSS8402DW, Q161 BSS8402DW, Q162 BSS8402DW, Q163 BSS8402DW, Q164 BSS8402DW, Q165 BSS8402DW, Q166 BSS8402DW, Q167 BSS8402DW, Q168 BSS8402DW, Q169 BSS8402DW, Q17 BSS8402DW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

Commit message: routed adder traces
Parts:
- removed R1: 470k, Resistor_SMD:R_0603_1608Metric_Pad1.05x0.95mm_HandSolder
- J1: value Conn_02x20_Odd_Even -> Conn_02x31_Top_Bottom; footprint Connector_PinHeader_2.54mm:PinHeader_2x20_P2.54mm_Vertical -> Tritium:BUS_AT_8bit
- moved J1 80.3 mm to (268.6, 54.0)
- moved Q3 39.8 mm to (31.8, 126.4), turned to 0 degrees
- moved Q5 35.4 mm to (238.1, 120.6), turned to 0 degrees
- moved R6 34.3 mm to (241.9, 121.9), turned to 180 degrees
- moved R528 33.3 mm to (261.0, 121.9), turned to 180 degrees
- moved Q348 32.6 mm to (35.6, 126.4), turned to 0 degrees
- moved R439 31.3 mm to (241.9, 120.0), turned to 0 degrees
- moved R452 31.2 mm to (249.6, 121.9), turned to 180 degrees
- moved Q350 30.7 mm to (245.7, 120.7), turned to 0 degrees
- moved R529 30.5 mm to (261.0, 120.0), turned to 0 degrees
- moved Q417 30.0 mm to (257.2, 120.7), turned to 0 degrees
- moved Q4 29.9 mm to (238.1, 115.6), turned to 0 degrees
- moved Q412 29.2 mm to (253.4, 120.7), turned to 0 degrees
- moved R517 28.1 mm to (249.6, 120.0), turned to 0 degrees
- moved Q1 28.1 mm to (31.8, 130.2), turned to 0 degrees
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Connections:
- net /Sheet712017E4/CarryIn renamed /adder/CarryIn
- net /Sheet712017E4/Vdd renamed /adder/Vdd
- net /Sheet712017E4/Vss renamed /adder/Vss
- net /sheet5FF29CD3/Vdd renamed /consensus/Vdd
- net /sheet5FF29CD3/Vss renamed /consensus/Vss
- net /sheet72A2BAFF/Vdd renamed /compare/Vdd
- net /sheet72A2BAFF/Vss renamed /compare/Vss
- net /sheet730CCE4E/Vdd renamed /min/Vdd
- net /sheet730CCE4E/Vss renamed /min/Vss
- net /sheet730D27DE/Vdd renamed /max/Vdd
- net /sheet730D27DE/Vss renamed /max/Vss
- net /sheet730E02CF/Vdd renamed /any/Vdd
- net /sheet730E02CF/Vss renamed /any/Vss
- net /sheet730E02D0/Vdd renamed /inverter/Vdd
- net /sheet730E02D0/Vss renamed /inverter/Vss
- net /sheet730EC5B7/Vdd renamed /sign/Vdd
- net /sheet730EC5B7/Vss renamed /sign/Vss
- J1 pad 1: A0 -> R8
- J1 pad 10: R1 -> Net-(J1-Pad10)
- J1 pad 11: A5 -> Net-(J1-Pad11)
- J1 pad 12: R2 -> Net-(J1-Pad12)
- J1 pad 13: A6 -> Net-(J1-Pad13)
- J1 pad 14: R3 -> Net-(J1-Pad14)
- J1 pad 15: A7 -> Net-(J1-Pad15)
- J1 pad 16: R4 -> Net-(J1-Pad16)
- J1 pad 17: A8 -> Net-(J1-Pad17)
- J1 pad 18: R5 -> Net-(J1-Pad18)
- J1 pad 19: B0 -> Vdd
- J1 pad 2: OutputEnable -> R7
- J1 pad 20: R6 -> GND
- J1 pad 21: B1 -> Vss
- J1 pad 22: R7 -> Net-(J1-Pad22)
- J1 pad 23: B2 -> Net-(J1-Pad23)
- J1 pad 24: R8 -> Net-(J1-Pad24)
- J1 pad 25: B3 -> Net-(J1-Pad25)
- J1 pad 27: B4 -> Net-(J1-Pad27)
- J1 pad 29: B5 -> Net-(J1-Pad29)
- J1 pad 3: A1 -> R6
- J1 pad 30: Net-(J1-Pad30) -> CarryIn
- J1 pad 31: B6 -> CarryOut
- J1 pad 32: Net-(J1-Pad32) -> A8
- J1 pad 33: B7 -> A7
- J1 pad 34: Net-(J1-Pad34) -> A6
- J1 pad 35: B8 -> A5
- J1 pad 36: Vdd -> A4
- J1 pad 37: CarryIn -> A3
- J1 pad 38: GND -> A2
- J1 pad 39: CarryOut -> A1
- J1 pad 4: Fn0 -> R5
- J1 pad 40: Vss -> A0
- J1 pad 5: A2 -> R4
- J1 pad 6: Fn1 -> R3
- J1 pad 7: A3 -> R2
- J1 pad 8: R0 -> R1
- J1 pad 9: A4 -> R0
Routing:
- net /adder/Vdd: track 0.00 -> 1096.6 mm, vias 0 -> 136
- net /adder/Vss: track 0.00 -> 155.8 mm, vias 0 -> 141
- net Net-(Q146-Pad2): track 0.00 -> 80.6 mm, vias 0 -> 3
- net Net-(Q80-Pad2): track 0.00 -> 78.7 mm, vias 0 -> 3
- net Net-(Q79-Pad2): track 0.00 -> 78.7 mm, vias 0 -> 3
- net Net-(Q78-Pad2): track 0.00 -> 78.7 mm, vias 0 -> 3
- net Net-(Q145-Pad2): track 0.00 -> 78.7 mm, vias 0 -> 3
- net Net-(Q14-Pad2): track 0.00 -> 78.7 mm, vias 0 -> 3
- net Net-(Q144-Pad2): track 0.00 -> 78.7 mm, vias 0 -> 3
- net Net-(Q13-Pad2): track 0.00 -> 78.3 mm, vias 0 -> 3
- net Net-(Q152-Pad2): track 0.00 -> 65.6 mm, vias 0 -> 2
- net Net-(Q151-Pad2): track 0.00 -> 65.6 mm, vias 0 -> 2
- net Net-(Q150-Pad2): track 0.00 -> 65.6 mm, vias 0 -> 2
- net Net-(Q137-Pad2): track 0.00 -> 65.6 mm, vias 0 -> 2
- net Net-(Q136-Pad2): track 0.00 -> 65.6 mm, vias 0 -> 2
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- added copper zone on B.Cu, net /adder/Vss
- added copper zone on B.Cu, net Vss
Other:
- board size 240 x 80.6 mm -> 247.7 x 81.3 mm
- board text added: "Function decoder"
- board text added: "Tritium-9 Arithmetic Logic Unit rev.0"
