File: pcbs/alu/rev.0/alu.kicad_pcb (KiCad board)
At the start: 2 copper layers, 247.7 x 81.3 mm, 1037 parts, among them J1 Conn_02x31_Top_Bottom, Q1 BSS8402DW, Q10 BSS8402DW, Q100 BSS8402DW, Q101 BSS8402DW, Q102 BSS8402DW, Q103 BSS8402DW, Q104 BSS8402DW, Q105 BSS8402DW, Q106 BSS8402DW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

Commit message: bss84 drain and source flipped
Connections:
- Q1 pad 6: Net-(Q1-Pad4) -> Net-(Q1-Pad3)
- Q10 pad 3: /adder/Vdd -> Net-(Q10-Pad3)
- Q10 pad 4: Net-(Q10-Pad4) -> /adder/Vdd
- Q102 pad 3: /adder/Vdd -> Net-(Q102-Pad3)
- Q102 pad 4: Net-(Q102-Pad4) -> /adder/Vdd
- Q103 pad 3: /adder/Vdd -> Net-(Q103-Pad3)
- Q103 pad 4: Net-(Q103-Pad4) -> /adder/Vdd
- Q104 pad 3: /adder/Vdd -> Net-(Q104-Pad3)
- Q104 pad 4: Net-(Q104-Pad4) -> /adder/Vdd
- Q105 pad 3: /adder/Vdd -> Net-(Q105-Pad3)
- Q105 pad 4: Net-(Q105-Pad4) -> /adder/Vdd
- Q106 pad 3: /adder/Vdd -> Net-(Q106-Pad3)
- Q106 pad 4: Net-(Q106-Pad4) -> /adder/Vdd
- Q107 pad 3: /adder/Vdd -> Net-(Q107-Pad3)
- Q107 pad 4: Net-(Q107-Pad4) -> /adder/Vdd
- Q108 pad 3: /adder/Vdd -> Net-(Q103-Pad3)
- Q108 pad 4: Net-(Q103-Pad4) -> /adder/Vdd
- Q109 pad 3: /adder/Vdd -> Net-(Q105-Pad3)
- Q109 pad 4: Net-(Q105-Pad4) -> /adder/Vdd
- Q11 pad 3: /adder/Vdd -> Net-(Q11-Pad3)
- Q11 pad 4: Net-(Q11-Pad4) -> /adder/Vdd
- Q110 pad 3: /adder/Vdd -> Net-(Q107-Pad3)
- Q110 pad 4: Net-(Q107-Pad4) -> /adder/Vdd
- Q111 pad 3: Net-(Q102-Pad4) -> Net-(Q111-Pad3)
- Q111 pad 4: Net-(Q111-Pad4) -> Net-(Q102-Pad3)
- Q112 pad 3: Net-(Q104-Pad4) -> Net-(Q112-Pad3)
- Q112 pad 4: Net-(Q112-Pad4) -> Net-(Q104-Pad3)
- Q113 pad 3: Net-(Q106-Pad4) -> Net-(Q113-Pad3)
- Q113 pad 4: Net-(Q113-Pad4) -> Net-(Q106-Pad3)
- Q114 pad 3: /adder/Vdd -> Net-(Q114-Pad3)
- Q114 pad 4: Net-(Q114-Pad4) -> /adder/Vdd
- Q115 pad 3: /adder/Vdd -> Net-(Q115-Pad3)
- Q115 pad 4: Net-(Q115-Pad4) -> /adder/Vdd
- Q116 pad 3: /adder/Vdd -> Net-(Q116-Pad3)
- Q116 pad 4: Net-(Q116-Pad4) -> /adder/Vdd
- Q117 pad 3: /adder/Vdd -> Net-(Q117-Pad3)
- Q117 pad 4: Net-(Q117-Pad4) -> /adder/Vdd
- Q118 pad 3: /adder/Vdd -> Net-(Q118-Pad3)
- Q118 pad 4: Net-(Q118-Pad4) -> /adder/Vdd
- Q119 pad 3: /adder/Vdd -> Net-(Q119-Pad3)
- Q119 pad 4: Net-(Q119-Pad4) -> /adder/Vdd
- Q12 pad 3: /adder/Vdd -> Net-(Q12-Pad3)
- Q12 pad 4: Net-(Q12-Pad4) -> /adder/Vdd
- Q120 pad 3: Net-(Q117-Pad4) -> Net-(Q120-Pad3)
- Q120 pad 4: Net-(Q120-Pad4) -> Net-(Q117-Pad3)
- Q121 pad 3: Net-(Q118-Pad4) -> Net-(Q121-Pad3)
- Q121 pad 4: Net-(Q121-Pad4) -> Net-(Q118-Pad3)
- Q122 pad 3: Net-(Q119-Pad4) -> Net-(Q122-Pad3)
- Q122 pad 4: Net-(Q122-Pad4) -> Net-(Q119-Pad3)
- Q123 pad 3: /adder/Vdd -> Net-(Q123-Pad3)
- Q123 pad 4: Net-(Q123-Pad4) -> /adder/Vdd
- Q124 pad 3: /adder/Vdd -> Net-(Q124-Pad3)
- Q124 pad 4: Net-(Q124-Pad4) -> /adder/Vdd
- Q125 pad 3: /adder/Vdd -> Net-(Q125-Pad3)
- Q125 pad 4: Net-(Q125-Pad4) -> /adder/Vdd
- Q126 pad 3: /adder/Vdd -> Net-(Q126-Pad3)
- Q126 pad 4: Net-(Q126-Pad4) -> /adder/Vdd
- Q127 pad 3: /adder/Vdd -> Net-(Q127-Pad3)
- Q127 pad 4: Net-(Q127-Pad4) -> /adder/Vdd
- Q128 pad 3: /adder/Vdd -> Net-(Q128-Pad3)
- Q128 pad 4: Net-(Q128-Pad4) -> /adder/Vdd
- Q129 pad 3: Net-(Q126-Pad4) -> Net-(Q129-Pad3)
- Q129 pad 4: Net-(Q129-Pad4) -> Net-(Q126-Pad3)
- Q13 pad 3: /adder/Vdd -> Net-(Q13-Pad3)
- Q13 pad 4: Net-(Q13-Pad4) -> /adder/Vdd
- Q130 pad 3: Net-(Q127-Pad4) -> Net-(Q130-Pad3)
- Q130 pad 4: Net-(Q130-Pad4) -> Net-(Q127-Pad3)
- Q131 pad 3: Net-(Q128-Pad4) -> Net-(Q131-Pad3)
- Q131 pad 4: Net-(Q131-Pad4) -> Net-(Q128-Pad3)
- Q132 pad 3: /adder/Vdd -> Net-(Q132-Pad3)
- Q132 pad 4: Net-(Q132-Pad4) -> /adder/Vdd
- Q133 pad 3: /adder/Vdd -> Net-(Q133-Pad3)
- Q133 pad 4: Net-(Q133-Pad4) -> /adder/Vdd
- Q134 pad 3: /adder/Vdd -> Net-(Q134-Pad3)
- Q134 pad 4: Net-(Q134-Pad4) -> /adder/Vdd
- Q135 pad 3: Net-(Q132-Pad4) -> Net-(Q135-Pad3)
- Q135 pad 4: Net-(Q135-Pad4) -> Net-(Q132-Pad3)
- Q136 pad 3: Net-(Q133-Pad4) -> Net-(Q136-Pad3)
- Q136 pad 4: Net-(Q136-Pad4) -> Net-(Q133-Pad3)
- Q137 pad 3: Net-(Q134-Pad4) -> Net-(Q137-Pad3)
- Q137 pad 4: Net-(Q137-Pad4) -> Net-(Q134-Pad3)
- Q138 pad 3: /adder/Vdd -> Net-(Q138-Pad3)
- Q138 pad 4: Net-(Q138-Pad4) -> /adder/Vdd
- Q139 pad 3: /adder/Vdd -> Net-(Q139-Pad3)
- Q139 pad 4: Net-(Q139-Pad4) -> /adder/Vdd
- Q14 pad 3: /adder/Vdd -> Net-(Q11-Pad3)
- Q14 pad 4: Net-(Q11-Pad4) -> /adder/Vdd
- Q140 pad 3: /adder/Vdd -> Net-(Q140-Pad3)
- Q140 pad 4: Net-(Q140-Pad4) -> /adder/Vdd
- Q141 pad 3: /adder/Vdd -> Net-(Q141-Pad3)
- Q141 pad 4: Net-(Q141-Pad4) -> /adder/Vdd
- Q142 pad 3: /adder/Vdd -> Net-(Q142-Pad3)
- Q142 pad 4: Net-(Q142-Pad4) -> /adder/Vdd
- Q143 pad 3: /adder/Vdd -> Net-(Q143-Pad3)
- Q143 pad 4: Net-(Q143-Pad4) -> /adder/Vdd
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Routing:
- net /adder/Vdd: track 1096.6 -> 0.00 mm, vias 136 -> 0
- net /adder/Vss: track 155.8 -> 0.00 mm, vias 141 -> 0
- net Net-(Q146-Pad2): track 80.6 -> 0.00 mm, vias 3 -> 0
- net Net-(Q80-Pad2): track 78.7 -> 0.00 mm, vias 3 -> 0
- net Net-(Q79-Pad2): track 78.7 -> 0.00 mm, vias 3 -> 0
- net Net-(Q78-Pad2): track 78.7 -> 0.00 mm, vias 3 -> 0
- net Net-(Q145-Pad2): track 78.7 -> 0.00 mm, vias 3 -> 0
- net Net-(Q14-Pad2): track 78.7 -> 0.00 mm, vias 3 -> 0
- net Net-(Q144-Pad2): track 78.7 -> 0.00 mm, vias 3 -> 0
- net Net-(Q13-Pad2): track 78.3 -> 0.00 mm, vias 3 -> 0
- net Net-(Q152-Pad2): track 65.6 -> 0.00 mm, vias 2 -> 0
- net Net-(Q151-Pad2): track 65.6 -> 0.00 mm, vias 2 -> 0
- net Net-(Q150-Pad2): track 65.6 -> 0.00 mm, vias 2 -> 0
- net Net-(Q137-Pad2): track 65.6 -> 0.00 mm, vias 2 -> 0
- net Net-(Q136-Pad2): track 65.6 -> 0.00 mm, vias 2 -> 0
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- removed copper zone on B.Cu, net /adder/Vss
- removed copper zone on B.Cu, net Vss
Other:
- board text removed: "Adder Instruction: (add) Add | A + B Instruction: (addc) Add with carry | A + B + C"
- board text removed: "Any Instruction: (any) Ternary any"
- board text removed: "Comparer Instruction: (cmp) Tritwise compare i: A < B | 0: A == B | 1: A > B"
- board text removed: "Consensus Instruction: (cons) Ternary consensus"
- board text removed: "Function decoder"
- board text removed: "Inverter Instruction: (inv) Ternary invert !A"
- board text removed: "Maximum Instruction: (max) Ternary maximum"
- board text removed: "Minimum Instruction: (min) Ternary minimum"
- board text removed: "Sign Instruction: (sign) Ternary sign i: A < 0 0: A == 0 1: A > 0"
- board text removed: "Tritium-9 Arithmetic Logic Unit rev.0"
