File: pcbs/gates/antimax/rev.2/antimax.kicad_pcb (KiCad board)
At the start: 2 copper layers, 10.2 x 7.6 mm, 6 parts, among them J1 Conn_01x03, J2 Conn_01x03, Q1 BSS8402DW, Q2 BSS8402DW

Commit message: added gate name to rev.2 pcbs and added clip gate
Other:
- board text added: "antimax gate"
- board text added: "rev.2"
Changed lines of the file:
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@@
   (general
     (thickness 1.6)
-    (drawings 4)
+    (drawings 6)
     (tracks 57)
     (zones 0)
@@
       (effects (font (size 1 1) (thickness 0.15)))
     )
+    (fp_line (start -0.8 0.4) (end -0.8 -0.4) (layer F.Fab) (width 0.1))
+    (fp_line (start -0.8 -0.4) (end 0.8 -0.4) (layer F.Fab) (width 0.1))
+    (fp_line (start 0.8 -0.4) (end 0.8 0.4) (layer F.Fab) (width 0.1))
+    (fp_line (start 0.8 0.4) (end -0.8 0.4) (layer F.Fab) (width 0.1))
+    (fp_line (start -0.171267 -0.51) (end 0.171267 -0.51) (layer F.SilkS) (width 0.12))
+    (fp_line (start -0.171267 0.51) (end 0.171267 0.51) (layer F.SilkS) (width 0.12))
+    (fp_line (start -1.65 0.73) (end -1.65 -0.73) (layer F.CrtYd) (width 0.05))
+    (fp_line (start -1.65 -0.73) (end 1.65 -0.73) (layer F.CrtYd) (width 0.05))
+    (fp_line (start 1.65 -0.73) (end 1.65 0.73) (layer F.CrtYd) (width 0.05))
     (fp_line (start 1.65 0.73) (end -1.65 0.73) (layer F.CrtYd) (width 0.05))
-    (fp_line (start 1.65 -0.73) (end 1.65 0.73) (layer F.CrtYd) (width 0.05))
-    (fp_line (start -1.65 -0.73) (end 1.65 -0.73) (layer F.CrtYd) (width 0.05))
-    (fp_line (start -1.65 0.73) (end -1.65 -0.73) (layer F.CrtYd) (width 0.05))
-    (fp_line (start -0.171267 0.51) (end 0.171267 0.51) (layer F.SilkS) (width 0.12))
-    (fp_line (start -0.171267 -0.51) (end 0.171267 -0.51) (layer F.SilkS) (width 0.12))
-    (fp_line (start 0.8 0.4) (end -0.8 0.4) (layer F.Fab) (width 0.1))
-    (fp_line (start 0.8 -0.4) (end 0.8 0.4) (layer F.Fab) (width 0.1))
-    (fp_line (start -0.8 -0.4) (end 0.8 -0.4) (layer F.Fab) (width 0.1))
-    (fp_line (start -0.8 0.4) (end -0.8 -0.4) (layer F.Fab) (width 0.1))
     (fp_text user %R (at 0 0) (layer F.Fab)
       (effects (font (size 0.4 0.4) (thickness 0.06)))
@@
       (effects (font (size 1 1) (thickness 0.15)))
     )
+    (fp_line (start -0.8 0.4) (end -0.8 -0.4) (layer F.Fab) (width 0.1))
+    (fp_line (start -0.8 -0.4) (end 0.8 -0.4) (layer F.Fab) (width 0.1))
+    (fp_line (start 0.8 -0.4) (end 0.8 0.4) (layer F.Fab) (width 0.1))
+    (fp_line (start 0.8 0.4) (end -0.8 0.4) (layer F.Fab) (width 0.1))
+    (fp_line (start -0.171267 -0.51) (end 0.171267 -0.51) (layer F.SilkS) (width 0.12))
+    (fp_line (start -0.171267 0.51) (end 0.171267 0.51) (layer F.SilkS) (width 0.12))
+    (fp_line (start -1.65 0.73) (end -1.65 -0.73) (layer F.CrtYd) (width 0.05))
+    (fp_line (start -1.65 -0.73) (end 1.65 -0.73) (layer F.CrtYd) (width 0.05))
+    (fp_line (start 1.65 -0.73) (end 1.65 0.73) (layer F.CrtYd) (width 0.05))
     (fp_line (start 1.65 0.73) (end -1.65 0.73) (layer F.CrtYd) (width 0.05))
-    (fp_line (start 1.65 -0.73) (end 1.65 0.73) (layer F.CrtYd) (width 0.05))
-    (fp_line (start -1.65 -0.73) (end 1.65 -0.73) (layer F.CrtYd) (width 0.05))
-    (fp_line (start -1.65 0.73) (end -1.65 -0.73) (layer F.CrtYd) (width 0.05))
-    (fp_line (start -0.171267 0.51) (end 0.171267 0.51) (layer F.SilkS) (width 0.12))
-    (fp_line (start -0.171267 -0.51) (end 0.171267 -0.51) (layer F.SilkS) (width 0.12))
-    (fp_line (start 0.8 0.4) (end -0.8 0.4) (layer F.Fab) (width 0.1))
-    (fp_line (start 0.8 -0.4) (end 0.8 0.4) (layer F.Fab) (width 0.1))
-    (fp_line (start -0.8 -0.4) (end 0.8 -0.4) (layer F.Fab) (width 0.1))
-    (fp_line (start -0.8 0.4) (end -0.8 -0.4) (layer F.Fab) (width 0.1))
     (fp_text user %R (at 0 0) (layer F.Fab)
       (effects (font (size 0.4 0.4) (thickness 0.06)))
@@
       (effects (font (size 1 1) (thickness 0.15)))
     )
+    (fp_line (start 0.7 -1.16) (end -1.2 -1.16) (layer F.SilkS) (width 0.12))
+    (fp_line (start -0.7 1.16) (end 0.7 1.16) (layer F.SilkS) (width 0.12))
+    (fp_line (start 1.6 1.4) (end 1.6 -1.4) (layer F.CrtYd) (width 0.05))
+    (fp_line (start -1.6 -1.4) (end -1.6 1.4) (layer F.CrtYd) (width 0.05))
+    (fp_line (start -1.6 -1.4) (end 1.6 -1.4) (layer F.CrtYd) (width 0.05))
+    (fp_line (start 0.675 -1.1) (end -0.175 -1.1) (layer F.Fab) (width 0.1))
+    (fp_line (start -0.675 -0.6) (end -0.675 1.1) (layer F.Fab) (width 0.1))
+    (fp_line (start -1.6 1.4) (end 1.6 1.4) (layer F.CrtYd) (width 0.05))
+    (fp_line (start 0.675 -1.1) (end 0.675 1.1) (layer F.Fab) (width 0.1))
+    (fp_line (start 0.675 1.1) (end -0.675 1.1) (layer F.Fab) (width 0.1))
     (fp_line (start -0.175 -1.1) (end -0.675 -0.6) (layer F.Fab) (width 0.1))
-    (fp_line (start 0.675 1.1) (end -0.675 1.1) (layer F.Fab) (width 0.1))
-    (fp_line (start 0.675 -1.1) (end 0.675 1.1) (layer F.Fab) (width 0.1))
-    (fp_line (start -1.6 1.4) (end 1.6 1.4) (layer F.CrtYd) (width 0.05))
-    (fp_line (start -0.675 -0.6) (end -0.675 1.1) (layer F.Fab) (width 0.1))
-    (fp_line (start 0.675 -1.1) (end -0.175 -1.1) (layer F.Fab) (width 0.1))
-    (fp_line (start -1.6 -1.4) (end 1.6 -1.4) (layer F.CrtYd) (width 0.05))
-    (fp_line (start -1.6 -1.4) (end -1.6 1.4) (layer F.CrtYd) (width 0.05))
-    (fp_line (start 1.6 1.4) (end 1.6 -1.4) (layer F.CrtYd) (width 0.05))
-    (fp_line (start -0.7 1.16) (end 0.7 1.16) (layer F.SilkS) (width 0.12))
-    (fp_line (start 0.7 -1.16) (end -1.2 -1.16) (layer F.SilkS) (width 0.12))
     (fp_text user %R (at 0 0 90) (layer F.Fab)
       (effects (font (size 0.5 0.5) (thickness 0.075)))
@@
       (effects (font (size 1 1) (thickness 0.15)))
     )
+    (fp_line (start 0.7 -1.16) (end -1.2 -1.16) (layer F.SilkS) (width 0.12))
+    (fp_line (start -0.7 1.16) (end 0.7 1.16) (layer F.SilkS) (width 0.12))
+    (fp_line (start 1.6 1.4) (end 1.6 -1.4) (layer F.CrtYd) (width 0.05))
+    (fp_line (start -1.6 -1.4) (end -1.6 1.4) (layer F.CrtYd) (width 0.05))
+    (fp_line (start -1.6 -1.4) (end 1.6 -1.4) (layer F.CrtYd) (width 0.05))
+    (fp_line (start 0.675 -1.1) (end -0.175 -1.1) (layer F.Fab) (width 0.1))
+    (fp_line (start -0.675 -0.6) (end -0.675 1.1) (layer F.Fab) (width 0.1))
+    (fp_line (start -1.6 1.4) (end 1.6 1.4) (layer F.CrtYd) (width 0.05))
+    (fp_line (start 0.675 -1.1) (end 0.675 1.1) (layer F.Fab) (width 0.1))
+    (fp_line (start 0.675 1.1) (end -0.675 1.1) (layer F.Fab) (width 0.1))
     (fp_line (start -0.175 -1.1) (end -0.675 -0.6) (layer F.Fab) (width 0.1))
-    (fp_line (start 0.675 1.1) (end -0.675 1.1) (layer F.Fab) (width 0.1))
-    (fp_line (start 0.675 -1.1) (end 0.675 1.1) (layer F.Fab) (width 0.1))
-    (fp_line (start -1.6 1.4) (end 1.6 1.4) (layer F.CrtYd) (width 0.05))
-    (fp_line (start -0.675 -0.6) (end -0.675 1.1) (layer F.Fab) (width 0.1))
-    (fp_line (start 0.675 -1.1) (end -0.175 -1.1) (layer F.Fab) (width 0.1))
-    (fp_line (start -1.6 -1.4) (end 1.6 -1.4) (layer F.CrtYd) (width 0.05))
-    (fp_line (start -1.6 -1.4) (end -1.6 1.4) (layer F.CrtYd) (width 0.05))
-    (fp_line (start 1.6 1.4) (end 1.6 -1.4) (layer F.CrtYd) (width 0.05))
-    (fp_line (start -0.7 1.16) (end 0.7 1.16) (layer F.SilkS) (width 0.12))
-    (fp_line (start 0.7 -1.16) (end -1.2 -1.16) (layer F.SilkS) (width 0.12))
     (fp_text user %R (at 0 0 90) (layer F.Fab)
       (effects (font (size 0.5 0.5) (thickness 0.075)))
@@
       (effects (font (size 1 1) (thickness 0.15)))
     )
+    (fp_line (start -1.27 -1.27) (end 0.635 -1.27) (layer F.Fab) (width 0.1))
+    (fp_line (start 0.635 -1.27) (end 1.27 -0.635) (layer F.Fab) (width 0.1))
+    (fp_line (start 1.27 -0.635) (end 1.27 6.35) (layer F.Fab) (width 0.1))
+    (fp_line (start 1.27 6.35) (end -1.27 6.35) (layer F.Fab) (width 0.1))
     (fp_line (start -1.27 6.35) (end -1.27 -1.27) (layer F.Fab) (width 0.1))
-    (fp_line (start 1.27 6.35) (end -1.27 6.35) (layer F.Fab) (width 0.1))
-    (fp_line (start 1.27 -0.635) (end 1.27 6.35) (layer F.Fab) (width 0.1))
-    (fp_line (start 0.635 -1.27) (end 1.27 -0.635) (layer F.Fab) (width 0.1))
-    (fp_line (start -1.27 -1.27) (end 0.635 -1.27) (layer F.Fab) (width 0.1))
     (fp_arc (start 0 0) (end 0 1.016) (angle -180) (layer F.SilkS) (width 0.12))
     (fp_text user %R (at 0 2.54 90) (layer F.Fab)
@@
       (effects (font (size 1 1) (thickness 0.15)))
     )
+    (fp_line (start -1.27 -1.27) (end 0.635 -1.27) (layer F.Fab) (width 0.1))
+    (fp_line (start 0.635 -1.27) (end 1.27 -0.635) (layer F.Fab) (width 0.1))
+    (fp_line (start 1.27 -0.635) (end 1.27 6.35) (layer F.Fab) (width 0.1))
+    (fp_line (start 1.27 6.35) (end -1.27 6.35) (layer F.Fab) (width 0.1))
     (fp_line (start -1.27 6.35) (end -1.27 -1.27) (layer F.Fab) (width 0.1))
-    (fp_line (start 1.27 6.35) (end -1.27 6.35) (layer F.Fab) (width 0.1))
-    (fp_line (start 1.27 -0.635) (end 1.27 6.35) (layer F.Fab) (width 0.1))
-    (fp_line (start 0.635 -1.27) (end 1.27 -0.635) (layer F.Fab) (width 0.1))
-    (fp_line (start -1.27 -1.27) (end 0.635 -1.27) (layer F.Fab) (width 0.1))
     (fp_arc (start 0 0) (end 0 1.016) (angle -180) (layer F.SilkS) (width 0.12))
     (fp_text user %R (at 0 2.54 90) (layer F.Fab)
@@
       (net 5 A))
   )
+  (gr_text rev.2 (at 110.744 64.008) (layer B.SilkS)
+    (effects (font (size 1 1) (thickness 0.15)) (justify mirror))
+  )
+  (gr_text "antimax\ngate\n\n" (at 110.744 59.436) (layer B.SilkS)
+    (effects (font (size 1 1) (thickness 0.15)) (justify mirror))
+  )
   (gr_line (start 115.57 57.15) (end 115.57 64.77) (layer Edge.Cuts) (width 0.1))
