File: pcbs/gates/inverter/rev.2/inverter.kicad_pcb (KiCad board)
At the start: 2 copper layers, 7.6 x 7.6 mm, 5 parts, among them J1 Conn_01x03, J2 Conn_01x03, Q1 BSS8402DW

Commit message: added gate name to rev.2 pcbs and added clip gate
Other:
- board text added: "inverter gate"
- board text added: "rev.2"
Changed lines of the file:
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@@
   (general
     (thickness 1.6)
-    (drawings 4)
+    (drawings 6)
     (tracks 42)
     (zones 0)
@@
       (effects (font (size 1 1) (thickness 0.15)))
     )
+    (fp_line (start 1.65 0.73) (end -1.65 0.73) (layer F.CrtYd) (width 0.05))
+    (fp_line (start 1.65 -0.73) (end 1.65 0.73) (layer F.CrtYd) (width 0.05))
+    (fp_line (start -1.65 -0.73) (end 1.65 -0.73) (layer F.CrtYd) (width 0.05))
+    (fp_line (start -1.65 0.73) (end -1.65 -0.73) (layer F.CrtYd) (width 0.05))
+    (fp_line (start -0.171267 0.51) (end 0.171267 0.51) (layer F.SilkS) (width 0.12))
+    (fp_line (start -0.171267 -0.51) (end 0.171267 -0.51) (layer F.SilkS) (width 0.12))
+    (fp_line (start 0.8 0.4) (end -0.8 0.4) (layer F.Fab) (width 0.1))
+    (fp_line (start 0.8 -0.4) (end 0.8 0.4) (layer F.Fab) (width 0.1))
+    (fp_line (start -0.8 -0.4) (end 0.8 -0.4) (layer F.Fab) (width 0.1))
+    (fp_line (start -0.8 0.4) (end -0.8 -0.4) (layer F.Fab) (width 0.1))
     (fp_text user %R (at 0 0) (layer F.Fab)
       (effects (font (size 0.4 0.4) (thickness 0.06)))
     )
-    (fp_line (start -0.8 0.4) (end -0.8 -0.4) (layer F.Fab) (width 0.1))
-    (fp_line (start -0.8 -0.4) (end 0.8 -0.4) (layer F.Fab) (width 0.1))
-    (fp_line (start 0.8 -0.4) (end 0.8 0.4) (layer F.Fab) (width 0.1))
-    (fp_line (start 0.8 0.4) (end -0.8 0.4) (layer F.Fab) (width 0.1))
-    (fp_line (start -0.171267 -0.51) (end 0.171267 -0.51) (layer F.SilkS) (width 0.12))
-    (fp_line (start -0.171267 0.51) (end 0.171267 0.51) (layer F.SilkS) (width 0.12))
-    (fp_line (start -1.65 0.73) (end -1.65 -0.73) (layer F.CrtYd) (width 0.05))
-    (fp_line (start -1.65 -0.73) (end 1.65 -0.73) (layer F.CrtYd) (width 0.05))
-    (fp_line (start 1.65 -0.73) (end 1.65 0.73) (layer F.CrtYd) (width 0.05))
-    (fp_line (start 1.65 0.73) (end -1.65 0.73) (layer F.CrtYd) (width 0.05))
     (pad 2 smd roundrect (at 0.875 0 180) (size 1.05 0.95) (layers F.Cu F.Paste F.Mask) (roundrect_rratio 0.25)
       (net 5 Nti))
@@
       (effects (font (size 1 1) (thickness 0.15)))
     )
+    (fp_line (start 1.65 0.73) (end -1.65 0.73) (layer F.CrtYd) (width 0.05))
+    (fp_line (start 1.65 -0.73) (end 1.65 0.73) (layer F.CrtYd) (width 0.05))
+    (fp_line (start -1.65 -0.73) (end 1.65 -0.73) (layer F.CrtYd) (width 0.05))
+    (fp_line (start -1.65 0.73) (end -1.65 -0.73) (layer F.CrtYd) (width 0.05))
+    (fp_line (start -0.171267 0.51) (end 0.171267 0.51) (layer F.SilkS) (width 0.12))
+    (fp_line (start -0.171267 -0.51) (end 0.171267 -0.51) (layer F.SilkS) (width 0.12))
+    (fp_line (start 0.8 0.4) (end -0.8 0.4) (layer F.Fab) (width 0.1))
+    (fp_line (start 0.8 -0.4) (end 0.8 0.4) (layer F.Fab) (width 0.1))
+    (fp_line (start -0.8 -0.4) (end 0.8 -0.4) (layer F.Fab) (width 0.1))
+    (fp_line (start -0.8 0.4) (end -0.8 -0.4) (layer F.Fab) (width 0.1))
     (fp_text user %R (at 0 0) (layer F.Fab)
       (effects (font (size 0.4 0.4) (thickness 0.06)))
     )
-    (fp_line (start -0.8 0.4) (end -0.8 -0.4) (layer F.Fab) (width 0.1))
-    (fp_line (start -0.8 -0.4) (end 0.8 -0.4) (layer F.Fab) (width 0.1))
-    (fp_line (start 0.8 -0.4) (end 0.8 0.4) (layer F.Fab) (width 0.1))
-    (fp_line (start 0.8 0.4) (end -0.8 0.4) (layer F.Fab) (width 0.1))
-    (fp_line (start -0.171267 -0.51) (end 0.171267 -0.51) (layer F.SilkS) (width 0.12))
-    (fp_line (start -0.171267 0.51) (end 0.171267 0.51) (layer F.SilkS) (width 0.12))
-    (fp_line (start -1.65 0.73) (end -1.65 -0.73) (layer F.CrtYd) (width 0.05))
-    (fp_line (start -1.65 -0.73) (end 1.65 -0.73) (layer F.CrtYd) (width 0.05))
-    (fp_line (start 1.65 -0.73) (end 1.65 0.73) (layer F.CrtYd) (width 0.05))
-    (fp_line (start 1.65 0.73) (end -1.65 0.73) (layer F.CrtYd) (width 0.05))
     (pad 2 smd roundrect (at 0.875 0) (size 1.05 0.95) (layers F.Cu F.Paste F.Mask) (roundrect_rratio 0.25)
       (net 1 Out))
@@
       (effects (font (size 1 1) (thickness 0.15)))
     )
+    (fp_line (start -0.175 -1.1) (end -0.675 -0.6) (layer F.Fab) (width 0.1))
+    (fp_line (start 0.675 1.1) (end -0.675 1.1) (layer F.Fab) (width 0.1))
+    (fp_line (start 0.675 -1.1) (end 0.675 1.1) (layer F.Fab) (width 0.1))
+    (fp_line (start -1.6 1.4) (end 1.6 1.4) (layer F.CrtYd) (width 0.05))
+    (fp_line (start -0.675 -0.6) (end -0.675 1.1) (layer F.Fab) (width 0.1))
+    (fp_line (start 0.675 -1.1) (end -0.175 -1.1) (layer F.Fab) (width 0.1))
+    (fp_line (start -1.6 -1.4) (end 1.6 -1.4) (layer F.CrtYd) (width 0.05))
+    (fp_line (start -1.6 -1.4) (end -1.6 1.4) (layer F.CrtYd) (width 0.05))
+    (fp_line (start 1.6 1.4) (end 1.6 -1.4) (layer F.CrtYd) (width 0.05))
+    (fp_line (start -0.7 1.16) (end 0.7 1.16) (layer F.SilkS) (width 0.12))
+    (fp_line (start 0.7 -1.16) (end -1.2 -1.16) (layer F.SilkS) (width 0.12))
     (fp_text user %R (at 0 0 90) (layer F.Fab)
       (effects (font (size 0.5 0.5) (thickness 0.075)))
     )
-    (fp_line (start 0.7 -1.16) (end -1.2 -1.16) (layer F.SilkS) (width 0.12))
-    (fp_line (start -0.7 1.16) (end 0.7 1.16) (layer F.SilkS) (width 0.12))
-    (fp_line (start 1.6 1.4) (end 1.6 -1.4) (layer F.CrtYd) (width 0.05))
-    (fp_line (start -1.6 -1.4) (end -1.6 1.4) (layer F.CrtYd) (width 0.05))
-    (fp_line (start -1.6 -1.4) (end 1.6 -1.4) (layer F.CrtYd) (width 0.05))
-    (fp_line (start 0.675 -1.1) (end -0.175 -1.1) (layer F.Fab) (width 0.1))
-    (fp_line (start -0.675 -0.6) (end -0.675 1.1) (layer F.Fab) (width 0.1))
-    (fp_line (start -1.6 1.4) (end 1.6 1.4) (layer F.CrtYd) (width 0.05))
-    (fp_line (start 0.675 -1.1) (end 0.675 1.1) (layer F.Fab) (width 0.1))
-    (fp_line (start 0.675 1.1) (end -0.675 1.1) (layer F.Fab) (width 0.1))
-    (fp_line (start -0.175 -1.1) (end -0.675 -0.6) (layer F.Fab) (width 0.1))
     (pad 6 smd rect (at 0.95 -0.65) (size 0.65 0.4) (layers F.Cu F.Paste F.Mask)
       (net 5 Nti))
@@
       (effects (font (size 1 1) (thickness 0.15)))
     )
+    (fp_line (start -1.27 6.35) (end -1.27 -1.27) (layer F.Fab) (width 0.1))
+    (fp_line (start 1.27 6.35) (end -1.27 6.35) (layer F.Fab) (width 0.1))
+    (fp_line (start 1.27 -0.635) (end 1.27 6.35) (layer F.Fab) (width 0.1))
+    (fp_line (start 0.635 -1.27) (end 1.27 -0.635) (layer F.Fab) (width 0.1))
+    (fp_line (start -1.27 -1.27) (end 0.635 -1.27) (layer F.Fab) (width 0.1))
     (fp_text user %R (at 0 2.54 90) (layer F.Fab)
       (effects (font (size 1 1) (thickness 0.15)))
     )
     (fp_arc (start 0 0) (end 0 1.016) (angle -180) (layer F.SilkS) (width 0.12))
-    (fp_line (start -1.27 -1.27) (end 0.635 -1.27) (layer F.Fab) (width 0.1))
-    (fp_line (start 0.635 -1.27) (end 1.27 -0.635) (layer F.Fab) (width 0.1))
-    (fp_line (start 1.27 -0.635) (end 1.27 6.35) (layer F.Fab) (width 0.1))
-    (fp_line (start 1.27 6.35) (end -1.27 6.35) (layer F.Fab) (width 0.1))
-    (fp_line (start -1.27 6.35) (end -1.27 -1.27) (layer F.Fab) (width 0.1))
     (pad 1 thru_hole oval (at 0 0) (size 1.7 1.7) (drill 1) (layers *.Cu *.Mask)
       (net 6 Pti))
@@
       (effects (font (size 1 1) (thickness 0.15)))
     )
+    (fp_line (start -1.27 -1.27) (end 0.635 -1.27) (layer F.Fab) (width 0.1))
+    (fp_line (start 0.635 -1.27) (end 1.27 -0.635) (layer F.Fab) (width 0.1))
+    (fp_line (start 1.27 -0.635) (end 1.27 6.35) (layer F.Fab) (width 0.1))
+    (fp_line (start 1.27 6.35) (end -1.27 6.35) (layer F.Fab) (width 0.1))
     (fp_line (start -1.27 6.35) (end -1.27 -1.27) (layer F.Fab) (width 0.1))
-    (fp_line (start 1.27 6.35) (end -1.27 6.35) (layer F.Fab) (width 0.1))
-    (fp_line (start 1.27 -0.635) (end 1.27 6.35) (layer F.Fab) (width 0.1))
-    (fp_line (start 0.635 -1.27) (end 1.27 -0.635) (layer F.Fab) (width 0.1))
-    (fp_line (start -1.27 -1.27) (end 0.635 -1.27) (layer F.Fab) (width 0.1))
     (fp_arc (start 0 0) (end 0 1.016) (angle -180) (layer F.SilkS) (width 0.12))
     (fp_text user %R (at 0 2.54 90) (layer F.Fab)
@@
       (net 3 Vdd))
   )
+  (gr_text rev.2 (at 97.028 58.928) (layer B.SilkS)
+    (effects (font (size 1 1) (thickness 0.15)) (justify mirror))
+  )
+  (gr_text "inverter\ngate" (at 97.028 53.848) (layer B.SilkS)
+    (effects (font (size 1 1) (thickness 0.15)) (justify mirror))
+  )
   (gr_line (start 100.965 52.07) (end 100.965 59.69) (layer Edge.Cuts) (width 0.1))
   (gr_line (start 93.345 52.07) (end 100.965 52.07) (layer Edge.Cuts) (width 0.1))
   (gr_line (start 93.345 59.69) (end 93.345 52.07) (layer Edge.Cuts) (width 0.1))
   (gr_line (start 100.965 59.69) (end 93.345 59.69) (layer Edge.Cuts) (width 0.1))
-  (via (at 99.06 55.5498) (size 0.8) (drill 0.4) (layers F.Cu B.Cu) (net 5))
-  (via (at 99.7204 55.0164) (size 0.8) (drill 0.4) (layers F.Cu B.Cu) (net 6))
   (segment (start 98.03 58.42) (end 98.555 58.42) (width 0.25) (layer F.Cu) (net 1))
   (segment (start 98.555 58.42) (end 100.965 56.01) (width 0.25) (layer F.Cu) (net 1))
@@
   (segment (start 93.42 55.955) (end 93.345 55.88) (width 0.25) (layer F.Cu) (net 4))
   (segment (start 96.205 55.955) (end 93.42 55.955) (width 0.25) (layer F.Cu) (net 4))
+  (via (at 99.06 55.5498) (size 0.8) (drill 0.4) (layers F.Cu B.Cu) (net 5))
   (segment (start 98.105 55.165) (end 96.28 53.34) (width 0.25) (layer F.Cu) (net 5))
   (segment (start 98.105 55.305) (end 98.105 55.165) (width 0.25) (layer F.Cu) (net 5))
@@
   (segment (start 99.06 56.515) (end 100.965 58.42) (width 0.25) (layer B.Cu) (net 5))
   (segment (start 99.06 55.5498) (end 99.06 56.515) (width 0.25) (layer B.Cu) (net 5))
+  (via (at 99.7204 55.0164) (size 0.8) (drill 0.4) (layers F.Cu B.Cu) (net 6))
   (segment (start 96.205 58.345) (end 96.28 58.42) (width 0.25) (layer F.Cu) (net 6))
   (segment (start 96.205 56.605) (end 96.205 58.345) (width 0.25) (layer F.Cu) (net 6))
