File: pcbs/gates/quadstate/rev.2/quadstate.kicad_pcb (KiCad board)
At the start: 2 copper layers, 10.2 x 13.3 mm, 10 parts, among them J1 Conn_01x03, J2 Conn_01x03, Q1 BSS8402DW, Q2 BSS8402DW, Q3 BSS8402DW, Q4 BSS8402DW

Commit message: added gate name to rev.2 pcbs and added clip gate
Other:
- board text added: "quadstate gate"
- board text added: "rev.2"
