File: kicad/gates/nquadstate/panel.kicad_pcb (KiCad board)
At the start: 2 copper layers, 100 x 100 mm, 1233 parts, among them J1 Conn_01x03, J2 Conn_01x03, Q1 BSS8402DW-7-F, Q2 BSS8402DW-7-F, Q3 BSS8402DW-7-F

Commit message: fixed sum logic gate schematic and simulation
Parts:
- removed the REF** at (20.0, 112.5) (x2)
- removed the REF** at (20.0, 17.5) (x2)
- removed the REF** at (110.0, 17.5) (x2)
- added REF**: Fiducial, Fiducial, B.Cu at (110.0, 17.5)
- added REF**: Fiducial, Fiducial, B.Cu at (20.0, 112.5)
- added REF**: Fiducial, Fiducial, B.Cu at (20.0, 17.5)
- added REF**: Fiducial, Fiducial, F.Cu at (20.0, 17.5)
- added REF**: Fiducial, Fiducial, F.Cu at (110.0, 17.5)
- added REF**: Fiducial, Fiducial, F.Cu at (20.0, 112.5)
Other:
- board text added: "Balanced Ternary Not Quadstate Gates"
- board text removed: "JLCJLCJLCJLC"
